Commit message: fix joints and controller

File: rov_description/urdf/truster.xacro (robot description, xacro)
@@ -231,8 +231,8 @@
         </inertial>
     </link>
-    <joint name="truster_vertical_01_to_helice" type="continuous">
+    <!-- <joint name="truster_vertical_01_to_helice" type="continuous">
         <parent link="truster_vertical_01"/>
         <child link="truster_helice_vertical_01"/>
-        <origin xyz="0.0 0.025 0.0" rpy="3.1416 0 0" />
+        <origin xyz="0.0 0.027 0.0" rpy="3.1416 0 0" />
         <axis xyz="0 1 0" />
     </joint>
@@ -240,5 +240,5 @@
         <parent link="truster_vertical_02"/>
         <child link="truster_helice_vertical_02"/>
-        <origin xyz="0.0 0.025 0.0" rpy="3.1416 0 0" />
+        <origin xyz="0.0 0.027 0.0" rpy="3.1416 0 0" />
         <axis xyz="0 1 0" />
     </joint>
@@ -246,5 +246,5 @@
         <parent link="truster_horiz_01"/>
         <child link="truster_helice_horiz_01"/>
-        <origin xyz="0.0 0.025 0.0" rpy="3.1416 0 0" />
+        <origin xyz="0.0 0.027 0.0" rpy="3.1416 0 0" />
         <axis xyz="0 1 0" />
     </joint>
@@ -252,5 +252,5 @@
         <parent link="truster_horiz_02"/>
         <child link="truster_helice_horiz_02"/>
-        <origin xyz="0.0 0.025 0.0" rpy="3.1416 0 0" />
+        <origin xyz="0.0 0.027 0.0" rpy="3.1416 0 0" />
         <axis xyz="0 1 0" />
     </joint>
@@ -258,5 +258,5 @@
         <parent link="truster_horiz_03"/>
         <child link="truster_helice_horiz_03"/>
-        <origin xyz="0.0 0.025 0.0" rpy="3.1416 0 0" />
+        <origin xyz="0.0 0.027 0.0" rpy="3.1416 0 0" />
         <axis xyz="0 1 0" />
     </joint>
@@ -264,5 +264,53 @@
         <parent link="truster_horiz_04"/>
         <child link="truster_helice_horiz_04"/>
-        <origin xyz="0.0 0.025 0.0" rpy="3.1416 0 0" />
+        <origin xyz="0.0 0.027 0.0" rpy="3.1416 0 0" />
+        <axis xyz="0 1 0" />
+    </joint> -->
+    <joint name="truster_vertical_01_to_helice" type="revolute">
+        <parent link="truster_vertical_01"/>
+        <child link="truster_helice_vertical_01"/>
+        <origin xyz="0.0 0.027 0.0" rpy="3.1416 0 0" />
+        <dynamics damping="0.0" friction="0.0" />
+        <limit upper="3.14" lower="-3.14" effort="6" velocity="0.5" />
+        <axis xyz="0 1 0" />
+    </joint>
+    <joint name="truster_vertical_02_to_helice" type="revolute">
+        <parent link="truster_vertical_02"/>
+        <child link="truster_helice_vertical_02"/>
+        <origin xyz="0.0 0.027 0.0" rpy="3.1416 0 0" />
+        <dynamics damping="0.0" friction="0.0" />
+        <limit upper="3.14" lower="-3.14" effort="6" velocity="0.5" />
+        <axis xyz="0 1 0" />
+    </joint>
+    <joint name="truster_horiz_01_to_helice" type="revolute">
+        <parent link="truster_horiz_01"/>
+        <child link="truster_helice_horiz_01"/>
+        <origin xyz="0.0 0.027 0.0" rpy="3.1416 0 0" />
+        <dynamics damping="0.0" friction="0.0" />
+        <limit upper="3.14" lower="-3.14" effort="6" velocity="0.5" />
+        <axis xyz="0 1 0" />
+    </joint>
+    <joint name="truster_horiz_02_to_helice" type="revolute">
+        <parent link="truster_horiz_02"/>
+        <child link="truster_helice_horiz_02"/>
+        <origin xyz="0.0 0.027 0.0" rpy="3.1416 0 0" />
+        <dynamics damping="0.0" friction="0.0" />
+        <limit upper="3.14" lower="-3.14" effort="6" velocity="0.5" />
+        <axis xyz="0 1 0" />
+    </joint>
+    <joint name="truster_horiz_03_to_helice" type="revolute">
+        <parent link="truster_horiz_03"/>
+        <child link="truster_helice_horiz_03"/>
+        <origin xyz="0.0 0.027 0.0" rpy="3.1416 0 0" />
+        <dynamics damping="0.0" friction="0.0" />
+        <limit upper="3.14" lower="-3.14" effort="6" velocity="0.5" />
+        <axis xyz="0 1 0" />
+    </joint>
+    <joint name="truster_horiz_04_to_helice" type="revolute">
+        <parent link="truster_horiz_04"/>
+        <child link="truster_helice_horiz_04"/>
+        <origin xyz="0.0 0.027 0.0" rpy="3.1416 0 0" />
+        <dynamics damping="0.0" friction="0.0" />
+        <limit upper="3.14" lower="-3.14" effort="6" velocity="0.5" />
         <axis xyz="0 1 0" />
     </joint>

File: rov_simulation/urdf/rov_simulation.xacro (robot description, xacro)
@@ -106,5 +106,5 @@
     <gazebo>
         <plugin name="gazebo_ros_control" filename="libgazebo_ros_control.so">
-            <legacyModeNS>true</legacyModeNS>
+            <!-- <legacyModeNS>true</legacyModeNS> -->
             <robotNamespace>/rov</robotNamespace>
             <robotSimType>gazebo_ros_control/DefaultRobotHWSim</robotSimType>

Commit message: change joint parameters and controllers joints

File: rov_description/urdf/truster.xacro (robot description, xacro)
@@ -231,5 +231,5 @@
         </inertial>
     </link>
-    <!-- <joint name="truster_vertical_01_to_helice" type="continuous">
+    <joint name="truster_vertical_01_to_helice" type="continuous">
         <parent link="truster_vertical_01"/>
         <child link="truster_helice_vertical_01"/>
@@ -266,6 +266,6 @@
         <origin xyz="0.0 0.027 0.0" rpy="3.1416 0 0" />
         <axis xyz="0 1 0" />
-    </joint> -->
-    <joint name="truster_vertical_01_to_helice" type="revolute">
+    </joint>
+    <!-- <joint name="truster_vertical_01_to_helice" type="revolute">
         <parent link="truster_vertical_01"/>
         <child link="truster_helice_vertical_01"/>
@@ -314,4 +314,4 @@
         <limit upper="3.14" lower="-3.14" effort="6" velocity="0.5" />
         <axis xyz="0 1 0" />
-    </joint>
+    </joint> -->
 </robot>

File: rov_simulation/urdf/rov_simulation.xacro (robot description, xacro)
@@ -167,3 +167,18 @@
     </sensor>
   </gazebo>
+    <!-- <gazebo>
+        <plugin name="skid_steer_drive_controller" filename="libgazebo_ros_skid_steer_drive.so">
+            <updateRate>100.0</updateRate>
+            <leftFrontJoint>left_base_mat_to_left_wheel_front</leftFrontJoint>
+            <rightFrontJoint>right_base_mat_to_right_wheel_front</rightFrontJoint>
+            <leftRearJoint>left_base_mat_to_left_wheel_back</leftRearJoint>
+            <rightRearJoint>right_base_mat_to_right_wheel_back</rightRearJoint>
+            <wheelSeparation>5.21395246</wheelSeparation>
+            <wheelDiameter>1.48103523</wheelDiameter>
+            <robotBaseFrame>base_link</robotBaseFrame>
+            <torque>2000000</torque>
+            <topicName>cmd_vel</topicName>
+            <broadcastTF>false</broadcastTF>
+        </plugin>
+    </gazebo> -->
 </robot>
